Commit message: fix

File: march_description/urdf/test_joint_rotational.xacro (robot description, xacro)
@@ -1,5 +1,5 @@
 <?xml version="1.0"?>
 <!-- Revolute-Revolute Manipulator -->
-<robot name="march" xmlns:xacro="http://www.ros.org/wiki/xacro">
+<robot name="rotational_joint" xmlns:xacro="http://www.ros.org/wiki/xacro">
     <!-- Switch between airgaiting or standing on the ground-->
     <!--Value set to: 'world' fixes the robot to the world-->
@@ -14,6 +14,6 @@
     <xacro:property name="bar_width" value="0.05"/>
     <xacro:property name="joint_buffer" value="${3*pi/180}"/> <!-- rad -->
-    <xacro:property name="joint_lower_limit" value="-0.5673"/> <!-- rad -->
-    <xacro:property name="joint_upper_limit" value="0.3549"/> <!-- rad -->
+    <xacro:property name="joint_lower_limit" value="-0.160925"/> <!-- rad --> <!--   0.741-->
+    <xacro:property name="joint_upper_limit" value="0.913349"/> <!-- rad --> <!--  0.919-->
     <xacro:property name="joint_effort_limit" value="21840"/> <!-- IU = 20 A -->
     <xacro:property name="joint_velocity_limit" value="2.0"/> <!-- rad/s -->
